File: robotic_hand_pcb_imu.kicad_sch (KiCad schematic)
At the start: 13 parts, among them U4 BNO085, Y3 32k768

Commit message: Add 5V buck regulator
Parts:
- renumbered C17 to C21, C18 to C22, C19 to C23, C20 to C24, C21 to C25, R8 to R10, R9 to R11, R5 to R7, R6 to R8, R7 to R9, U4 to U5
Changed lines of the file:
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@@
 		(shape input)
 		(at 72.39 76.2 180)
-		(fields_autoplaced yes)
 		(effects
 			(font
@@
 		(shape input)
 		(at 72.39 71.12 180)
-		(fields_autoplaced yes)
 		(effects
 			(font
@@
 		(shape input)
 		(at 115.57 68.58 0)
-		(fields_autoplaced yes)
 		(effects
 			(font
@@
 		(shape input)
 		(at 72.39 78.74 180)
-		(fields_autoplaced yes)
 		(effects
 			(font
@@
 		(shape input)
 		(at 53.34 63.5 180)
-		(fields_autoplaced yes)
 		(effects
 			(font
@@
 		(shape input)
 		(at 72.39 66.04 180)
-		(fields_autoplaced yes)
 		(effects
 			(font
@@
 		(shape input)
 		(at 72.39 73.66 180)
-		(fields_autoplaced yes)
 		(effects
 			(font
@@
 		(on_board yes)
 		(dnp no)
-		(property "Reference" "#PWR042"
+		(property "Reference" "#PWR049"
 			(at 182.88 67.31 0)
 			(effects
@@
 			(project "robotic_hand_pcb"
 				(path "/96df9010-a1f8-4419-aac0-9388de87cb21/f209e5e9-1726-454a-82e1-5fd492ecf1c3"
-					(reference "#PWR042")
+					(reference "#PWR049")
 					(unit 1)
 				)
@@
 		(on_board yes)
 		(dnp no)
-		(property "Reference" "C19"
+		(property "Reference" "C23"
 			(at 120.65 48.26 0)
 			(effects
@@
 			(project "robotic_hand_pcb"
 				(path "/96df9010-a1f8-4419-aac0-9388de87cb21/f209e5e9-1726-454a-82e1-5fd492ecf1c3"
-					(reference "C19")
+					(reference "C23")
 					(unit 1)
 				)
@@
 		(on_board yes)
 		(dnp no)
-		(property "Reference" "R8"
+		(property "Reference" "R10"
 			(at 171.704 67.31 0)
 			(effects
@@
 			(project "robotic_hand_pcb"
 				(path "/96df9010-a1f8-4419-aac0-9388de87cb21/f209e5e9-1726-454a-82e1-5fd492ecf1c3"
-					(reference "R8")
+					(reference "R10")
 					(unit 1)
 				)
@@
 		(dnp no)
 		(fields_autoplaced yes)
-		(property "Reference" "#PWR045"
+		(property "Reference" "#PWR052"
 			(at 87.63 105.41 0)
 			(effects
@@
 			(project "robotic_hand_pcb"
 				(path "/96df9010-a1f8-4419-aac0-9388de87cb21/f209e5e9-1726-454a-82e1-5fd492ecf1c3"
-					(reference "#PWR045")
+					(reference "#PWR052")
 					(unit 1)
 				)
@@
 		(on_board yes)
 		(dnp no)
-		(property "Reference" "R6"
+		(property "Reference" "R8"
 			(at 53.086 57.15 0)
 			(effects
@@
 			(project "robotic_hand_pcb"
 				(path "/96df9010-a1f8-4419-aac0-9388de87cb21/f209e5e9-1726-454a-82e1-5fd492ecf1c3"
-					(reference "R6")
+					(reference "R8")
 					(unit 1)
 				)
@@
 		(on_board yes)
 		(dnp no)
-		(property "Reference" "#PWR039"
+		(property "Reference" "#PWR046"
 			(at 162.56 58.42 0)
 			(effects
@@
 			(project "robotic_hand_pcb"
 				(path "/96df9010-a1f8-4419-aac0-9388de87cb21/f209e5e9-1726-454a-82e1-5fd492ecf1c3"
-					(reference "#PWR039")
+					(reference "#PWR046")
 					(unit 1)
 				)
@@
 		(dnp no)
 		(fields_autoplaced yes)
-		(property "Reference" "#PWR036"
+		(property "Reference" "#PWR043"
 			(at 106.68 49.53 0)
 			(effects
@@
 			(project "robotic_hand_pcb"
 				(path "/96df9010-a1f8-4419-aac0-9388de87cb21/f209e5e9-1726-454a-82e1-5fd492ecf1c3"
-					(reference "#PWR036")
+					(reference "#PWR043")
 					(unit 1)
 				)
@@
 		(on_board yes)
 		(dnp no)
-		(property "Reference" "#PWR037"
+		(property "Reference" "#PWR044"
 			(at 67.31 49.53 0)
 			(effects
@@
 			(project "robotic_hand_pcb"
 				(path "/96df9010-a1f8-4419-aac0-9388de87cb21/f209e5e9-1726-454a-82e1-5fd492ecf1c3"
-					(reference "#PWR037")
+					(reference "#PWR044")
 					(unit 1)
 				)
@@
 		(dnp no)
 		(fields_autoplaced yes)
-		(property "Reference" "#PWR044"
+		(property "Reference" "#PWR051"
 			(at 93.98 97.79 0)
 			(effects
@@
 			(project "robotic_hand_pcb"
 				(path "/96df9010-a1f8-4419-aac0-9388de87cb21/f209e5e9-1726-454a-82e1-5fd492ecf1c3"
-					(reference "#PWR044")
+					(reference "#PWR051")
 					(unit 1)
 				)
@@
 		(on_board yes)
 		(dnp no)
-		(property "Reference" "C20"
+		(property "Reference" "C24"
 			(at 138.43 48.26 0)
 			(effects
@@
 			(project "robotic_hand_pcb"
 				(path "/96df9010-a1f8-4419-aac0-9388de87cb21/f209e5e9-1726-454a-82e1-5fd492ecf1c3"
-					(reference "C20")
+					(reference "C24")
 					(unit 1)
 				)
@@
 		(on_board yes)
 		(dnp no)
-		(property "Reference" "R7"
+		(property "Reference" "R9"
 			(at 150.876 59.69 0)
 			(effects
@@
 			(project "robotic_hand_pcb"
 				(path "/96df9010-a1f8-4419-aac0-9388de87cb21/f209e5e9-1726-454a-82e1-5fd492ecf1c3"
-					(reference "R7")
+					(reference "R9")
 					(unit 1)
 				)
@@
 		(dnp no)
 		(fields_autoplaced yes)
-		(property "Reference" "#PWR040"
+		(property "Reference" "#PWR047"
 			(at 129.54 62.23 0)
 			(effects
@@
 			(project "robotic_hand_pcb"
 				(path "/96df9010-a1f8-4419-aac0-9388de87cb21/f209e5e9-1726-454a-82e1-5fd492ecf1c3"
-					(reference "#PWR040")
+					(reference "#PWR047")
 					(unit 1)
 				)
@@
 		(on_board yes)
 		(dnp no)
-		(property "Reference" "C18"
+		(property "Reference" "C22"
 			(at 109.22 35.56 0)
 			(effects
@@
 			(project "robotic_hand_pcb"
 				(path "/96df9010-a1f8-4419-aac0-9388de87cb21/f209e5e9-1726-454a-82e1-5fd492ecf1c3"
-					(reference "C18")
+					(reference "C22")
 					(unit 1)
 				)
@@
 		(on_board yes)
 		(dnp no)
-		(property "Reference" "U4"
+		(property "Reference" "U5"
 			(at 108.966 47.498 0)
 			(effects
@@
 			(project "robotic_hand_pcb"
 				(path "/96df9010-a1f8-4419-aac0-9388de87cb21/f209e5e9-1726-454a-82e1-5fd492ecf1c3"
-					(reference "U4")
+					(reference "U5")
 					(unit 1)
 				)
@@
 		(on_board yes)
 		(dnp no)
-		(property "Reference" "#PWR035"
+		(property "Reference" "#PWR042"
 			(at 106.68 34.29 0)
 			(effects
@@
 			(project "robotic_hand_pcb"
 				(path "/96df9010-a1f8-4419-aac0-9388de87cb21/f209e5e9-1726-454a-82e1-5fd492ecf1c3"
-					(reference "#PWR035")
+					(reference "#PWR042")
 					(unit 1)
 				)
@@
 		(dnp no)
 		(fields_autoplaced yes)
-		(property "Reference" "#PWR043"
+		(property "Reference" "#PWR050"
 			(at 152.4 72.39 0)
 			(effects
@@
 			(project "robotic_hand_pcb"
 				(path "/96df9010-a1f8-4419-aac0-9388de87cb21/f209e5e9-1726-454a-82e1-5fd492ecf1c3"
-					(reference "#PWR043")
+					(reference "#PWR050")
 					(unit 1)
 				)
@@
 		(on_board yes)
 		(dnp no)
-		(property "Reference" "C17"
+		(property "Reference" "C21"
 			(at 99.06 35.56 0)
 			(effects
@@
 			(project "robotic_hand_pcb"
 				(path "/96df9010-a1f8-4419-aac0-9388de87cb21/f209e5e9-1726-454a-82e1-5fd492ecf1c3"
-					(reference "C17")
+					(reference "C21")
 					(unit 1)
 				)
@@
 		(on_board yes)
 		(dnp no)
-		(property "Reference" "#PWR041"
+		(property "Reference" "#PWR048"
 			(at 170.18 67.31 0)
 			(effects
@@
 			(project "robotic_hand_pcb"
 				(path "/96df9010-a1f8-4419-aac0-9388de87cb21/f209e5e9-1726-454a-82e1-5fd492ecf1c3"
-					(reference "#PWR041")
+					(reference "#PWR048")
 					(unit 1)
 				)
@@
 		(on_board yes)
 		(dnp no)
-		(property "Reference" "R5"
+		(property "Reference" "R7"
 			(at 65.786 49.53 0)
 			(effects
@@
 			(project "robotic_hand_pcb"
 				(path "/96df9010-a1f8-4419-aac0-9388de87cb21/f209e5e9-1726-454a-82e1-5fd492ecf1c3"
-					(reference "R5")
+					(reference "R7")
 					(unit 1)
 				)
@@
 		(on_board yes)
 		(dnp no)
-		(property "Reference" "#PWR038"
+		(property "Reference" "#PWR045"
 			(at 54.61 57.15 0)
 			(effects
@@
 			(project "robotic_hand_pcb"
 				(path "/96df9010-a1f8-4419-aac0-9388de87cb21/f209e5e9-1726-454a-82e1-5fd492ecf1c3"
-					(reference "#PWR038")
+					(reference "#PWR045")
 					(unit 1)
 				)
@@
 		(on_board yes)
 		(dnp no)
-		(property "Reference" "R9"
+		(property "Reference" "R11"
 			(at 184.404 67.31 0)
 			(effects
@@
 			(project "robotic_hand_pcb"
 				(path "/96df9010-a1f8-4419-aac0-9388de87cb21/f209e5e9-1726-454a-82e1-5fd492ecf1c3"
-					(reference "R9")
+					(reference "R11")
 					(unit 1)
 				)
@@
 		(on_board yes)
 		(dnp no)
-		(property "Reference" "C21"
+		(property "Reference" "C25"
 			(at 83.82 92.7099 0)
 			(effects
@@
 			(project "robotic_hand_pcb"
 				(path "/96df9010-a1f8-4419-aac0-9388de87cb21/f209e5e9-1726-454a-82e1-5fd492ecf1c3"
-					(reference "C21")
-					(unit 1)
-				)
+					(reference "C25")
+					(unit 1)
+				)

Commit message: Update for WIP changes
Parts:
- renumbered C21 to C20, C22 to C21, C23 to C22, C24 to C23, C25 to C24, R11 to R10, R7 to R6, R8 to R7, R9 to R8, R10 to R9
Changed lines of the file:
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@@
 		(on_board yes)
 		(dnp no)
-		(property "Reference" "#PWR049"
+		(property "Reference" "#PWR043"
 			(at 182.88 67.31 0)
 			(effects
@@
 			(project "robotic_hand_pcb"
 				(path "/96df9010-a1f8-4419-aac0-9388de87cb21/f209e5e9-1726-454a-82e1-5fd492ecf1c3"
-					(reference "#PWR049")
+					(reference "#PWR043")
 					(unit 1)
 				)
@@
 		(on_board yes)
 		(dnp no)
-		(property "Reference" "C23"
+		(property "Reference" "C22"
 			(at 120.65 48.26 0)
 			(effects
@@
 			(project "robotic_hand_pcb"
 				(path "/96df9010-a1f8-4419-aac0-9388de87cb21/f209e5e9-1726-454a-82e1-5fd492ecf1c3"
-					(reference "C23")
+					(reference "C22")
 					(unit 1)
 				)
@@
 		(on_board yes)
 		(dnp no)
-		(property "Reference" "R10"
+		(property "Reference" "R9"
 			(at 171.704 67.31 0)
 			(effects
@@
 			(project "robotic_hand_pcb"
 				(path "/96df9010-a1f8-4419-aac0-9388de87cb21/f209e5e9-1726-454a-82e1-5fd492ecf1c3"
-					(reference "R10")
+					(reference "R9")
 					(unit 1)
 				)
@@
 		(dnp no)
 		(fields_autoplaced yes)
-		(property "Reference" "#PWR052"
+		(property "Reference" "#PWR046"
 			(at 87.63 105.41 0)
 			(effects
@@
 			(project "robotic_hand_pcb"
 				(path "/96df9010-a1f8-4419-aac0-9388de87cb21/f209e5e9-1726-454a-82e1-5fd492ecf1c3"
-					(reference "#PWR052")
+					(reference "#PWR046")
 					(unit 1)
 				)
@@
 		(on_board yes)
 		(dnp no)
-		(property "Reference" "R8"
+		(property "Reference" "R7"
 			(at 53.086 57.15 0)
 			(effects
@@
 			(project "robotic_hand_pcb"
 				(path "/96df9010-a1f8-4419-aac0-9388de87cb21/f209e5e9-1726-454a-82e1-5fd492ecf1c3"
-					(reference "R8")
+					(reference "R7")
 					(unit 1)
 				)
@@
 		(on_board yes)
 		(dnp no)
-		(property "Reference" "#PWR046"
+		(property "Reference" "#PWR040"
 			(at 162.56 58.42 0)
 			(effects
@@
 			(project "robotic_hand_pcb"
 				(path "/96df9010-a1f8-4419-aac0-9388de87cb21/f209e5e9-1726-454a-82e1-5fd492ecf1c3"
-					(reference "#PWR046")
+					(reference "#PWR040")
 					(unit 1)
 				)
@@
 		(dnp no)
 		(fields_autoplaced yes)
-		(property "Reference" "#PWR043"
+		(property "Reference" "#PWR037"
 			(at 106.68 49.53 0)
 			(effects
@@
 			(project "robotic_hand_pcb"
 				(path "/96df9010-a1f8-4419-aac0-9388de87cb21/f209e5e9-1726-454a-82e1-5fd492ecf1c3"
-					(reference "#PWR043")
+					(reference "#PWR037")
 					(unit 1)
 				)
@@
 		(on_board yes)
 		(dnp no)
-		(property "Reference" "#PWR044"
+		(property "Reference" "#PWR038"
 			(at 67.31 49.53 0)
 			(effects
@@
 			(project "robotic_hand_pcb"
 				(path "/96df9010-a1f8-4419-aac0-9388de87cb21/f209e5e9-1726-454a-82e1-5fd492ecf1c3"
-					(reference "#PWR044")
+					(reference "#PWR038")
 					(unit 1)
 				)
@@
 		(dnp no)
 		(fields_autoplaced yes)
-		(property "Reference" "#PWR051"
+		(property "Reference" "#PWR045"
 			(at 93.98 97.79 0)
 			(effects
@@
 			(project "robotic_hand_pcb"
 				(path "/96df9010-a1f8-4419-aac0-9388de87cb21/f209e5e9-1726-454a-82e1-5fd492ecf1c3"
-					(reference "#PWR051")
+					(reference "#PWR045")
 					(unit 1)
 				)
@@
 		(on_board yes)
 		(dnp no)
-		(property "Reference" "C24"
+		(property "Reference" "C23"
 			(at 138.43 48.26 0)
 			(effects
@@
 			(project "robotic_hand_pcb"
 				(path "/96df9010-a1f8-4419-aac0-9388de87cb21/f209e5e9-1726-454a-82e1-5fd492ecf1c3"
-					(reference "C24")
+					(reference "C23")
 					(unit 1)
 				)
@@
 		(on_board yes)
 		(dnp no)
-		(property "Reference" "R9"
+		(property "Reference" "R8"
 			(at 150.876 59.69 0)
 			(effects
@@
 			(project "robotic_hand_pcb"
 				(path "/96df9010-a1f8-4419-aac0-9388de87cb21/f209e5e9-1726-454a-82e1-5fd492ecf1c3"
-					(reference "R9")
+					(reference "R8")
 					(unit 1)
 				)
@@
 		(dnp no)
 		(fields_autoplaced yes)
-		(property "Reference" "#PWR047"
+		(property "Reference" "#PWR041"
 			(at 129.54 62.23 0)
 			(effects
@@
 			(project "robotic_hand_pcb"
 				(path "/96df9010-a1f8-4419-aac0-9388de87cb21/f209e5e9-1726-454a-82e1-5fd492ecf1c3"
-					(reference "#PWR047")
+					(reference "#PWR041")
 					(unit 1)
 				)
@@
 		(on_board yes)
 		(dnp no)
-		(property "Reference" "C22"
+		(property "Reference" "C21"
 			(at 109.22 35.56 0)
 			(effects
@@
 			(project "robotic_hand_pcb"
 				(path "/96df9010-a1f8-4419-aac0-9388de87cb21/f209e5e9-1726-454a-82e1-5fd492ecf1c3"
-					(reference "C22")
+					(reference "C21")
 					(unit 1)
 				)
@@
 		(on_board yes)
 		(dnp no)
-		(property "Reference" "#PWR042"
+		(property "Reference" "#PWR036"
 			(at 106.68 34.29 0)
 			(effects
@@
 			(project "robotic_hand_pcb"
 				(path "/96df9010-a1f8-4419-aac0-9388de87cb21/f209e5e9-1726-454a-82e1-5fd492ecf1c3"
-					(reference "#PWR042")
+					(reference "#PWR036")
 					(unit 1)
 				)
@@
 		(dnp no)
 		(fields_autoplaced yes)
-		(property "Reference" "#PWR050"
+		(property "Reference" "#PWR044"
 			(at 152.4 72.39 0)
 			(effects
@@
 			(project "robotic_hand_pcb"
 				(path "/96df9010-a1f8-4419-aac0-9388de87cb21/f209e5e9-1726-454a-82e1-5fd492ecf1c3"
-					(reference "#PWR050")
+					(reference "#PWR044")
 					(unit 1)
 				)
@@
 		(on_board yes)
 		(dnp no)
-		(property "Reference" "C21"
+		(property "Reference" "C20"
 			(at 99.06 35.56 0)
 			(effects
@@
 			(project "robotic_hand_pcb"
 				(path "/96df9010-a1f8-4419-aac0-9388de87cb21/f209e5e9-1726-454a-82e1-5fd492ecf1c3"
-					(reference "C21")
+					(reference "C20")
 					(unit 1)
 				)
@@
 		(on_board yes)
 		(dnp no)
-		(property "Reference" "#PWR048"
+		(property "Reference" "#PWR042"
 			(at 170.18 67.31 0)
 			(effects
@@
 			(project "robotic_hand_pcb"
 				(path "/96df9010-a1f8-4419-aac0-9388de87cb21/f209e5e9-1726-454a-82e1-5fd492ecf1c3"
-					(reference "#PWR048")
+					(reference "#PWR042")
 					(unit 1)
 				)
@@
 		(on_board yes)
 		(dnp no)
-		(property "Reference" "R7"
+		(property "Reference" "R6"
 			(at 65.786 49.53 0)
 			(effects
@@
 			(project "robotic_hand_pcb"
 				(path "/96df9010-a1f8-4419-aac0-9388de87cb21/f209e5e9-1726-454a-82e1-5fd492ecf1c3"
-					(reference "R7")
+					(reference "R6")
 					(unit 1)
 				)
@@
 		(on_board yes)
 		(dnp no)
-		(property "Reference" "#PWR045"
+		(property "Reference" "#PWR039"
 			(at 54.61 57.15 0)
 			(effects
@@
 			(project "robotic_hand_pcb"
 				(path "/96df9010-a1f8-4419-aac0-9388de87cb21/f209e5e9-1726-454a-82e1-5fd492ecf1c3"
-					(reference "#PWR045")
+					(reference "#PWR039")
 					(unit 1)
 				)
@@
 		(on_board yes)
 		(dnp no)
-		(property "Reference" "R11"
+		(property "Reference" "R10"
 			(at 184.404 67.31 0)
 			(effects
@@
 			(project "robotic_hand_pcb"
 				(path "/96df9010-a1f8-4419-aac0-9388de87cb21/f209e5e9-1726-454a-82e1-5fd492ecf1c3"
-					(reference "R11")
+					(reference "R10")
 					(unit 1)
 				)
@@
 		(on_board yes)
 		(dnp no)
-		(property "Reference" "C25"
+		(property "Reference" "C24"
 			(at 83.82 92.7099 0)
 			(effects
@@
 			(project "robotic_hand_pcb"
 				(path "/96df9010-a1f8-4419-aac0-9388de87cb21/f209e5e9-1726-454a-82e1-5fd492ecf1c3"
-					(reference "C25")
-					(unit 1)
-				)
+					(reference "C24")
+					(unit 1)
+				)

Commit message: Add WIP schematic changes
Parts:
- C20, C21, C22, C23, C24, R10, R6, R7, R8, R9, Y3: now not fitted
- U7: renamed from U5; now not fitted

Commit message: Pass ERC, update component_library
Parts:
- renumbered JP1 to JP2
Changed lines of the file:
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@@
 		(on_board yes)
 		(dnp no)
-		(property "Reference" "JP1"
+		(property "Reference" "JP2"
 			(at 157.48 60.96 0)
 			(effects
@@
 			(project "robotic_hand_pcb"
 				(path "/96df9010-a1f8-4419-aac0-9388de87cb21/f209e5e9-1726-454a-82e1-5fd492ecf1c3"
-					(reference "JP1")
+					(reference "JP2")
 					(unit 1)
 				)
