File: robotic_hand_pcb_analog.kicad_sch (KiCad schematic)
At the start: 26 parts, among them J10 A5, J11 A6, J12 A7, J6 A1, J7 A2, J8 A3, J9 A4, U10 ACS712xLCTR-05B, U11 ACS712xLCTR-05B, U12 ACS712xLCTR-05B, U13 ACS712xLCTR-05B, U8 ADS114S08, U9 ACS712xLCTR-05B

Commit message: Add WIP ADC routes
Connections:
- net ADC1: now also U8.19 (GPIO3/AIN11); no longer U8.3 (AIN4)
- net ADC10: now also U8.22 (GPIO0/AIN8); no longer U8.21 (GPIO1/AIN9)
- net ADC11: now also U8.21 (GPIO1/AIN9); no longer U8.20 (GPIO2/AIN10)
- net ADC12: now also U8.20 (GPIO2/AIN10); no longer U8.19 (GPIO3/AIN11)
- net ADC3: now also U8.7 (AIN0); no longer U8.5 (AIN2)
- net ADC5: now also U8.5 (AIN2); no longer U8.7 (AIN0)
- net ADC6: now also U8.3 (AIN4); no longer U8.2 (AIN5)
- net ADC7: now also U8.2 (AIN5); no longer U8.32 (REFP1_AIN6)
- net ADC8: now also U8.32 (REFP1_AIN6); no longer U8.31 (REFN1_AIN7)
- net ADC9: now also U8.31 (REFN1_AIN7); no longer U8.22 (GPIO0/AIN8)

Commit message: Initial full PCB design, pass DRC
Parts:
- renumbered J8 to J10, J9 to J11, J10 to J12, J11 to J13, J12 to J14, J6 to J8, J7 to J9

Commit message: Fix ADC IC decoupling
Parts:
- C25: value 100n -> 330n
Changed lines of the file:
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@@
 			)
 		)
-		(property "Value" "100n"
+		(property "Value" "330n"
 			(at 26.67 26.67 0)
 			(effects

Commit message: Utilize AINCOM
Connections:
- net GND: now also U8.1 (AINCOM)
- no-connect marks 3 -> 2
Changed lines of the file:
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@@
 		(at 22.86 41.91)
 	)
-	(no_connect
-		(at 22.86 46.99)
-	)
 	(wire
 		(pts
@@
 	(wire
 		(pts
+			(xy 21.59 48.26) (xy 21.59 46.99)
+		)
+		(stroke
+			(width 0)
+			(type default)
+		)
+	)
+	(wire
+		(pts
 			(xy 124.46 40.64) (xy 125.73 40.64)
 		)
@@
 	(wire
 		(pts
+			(xy 21.59 46.99) (xy 22.86 46.99)
+		)
+		(stroke
+			(width 0)
+			(type default)
+		)
+	)
+	(wire
+		(pts
 			(xy 52.07 154.94) (xy 52.07 156.21)
 		)
@@
 					(unit 1)
 				)
+			)
+		)
+	)
+	(symbol
+		(lib_id "power:GND")
+		(at 21.59 48.26 0)
+		(unit 1)
+		(exclude_from_sim no)
+		(in_bom yes)
+		(on_board yes)
+		(dnp no)
+		(fields_autoplaced yes)
+		(property "Reference" "#PWR0122"
+			(at 21.59 54.61 0)
+			(effects
+				(font
+					(size 1.27 1.27)
+				)
+				(hide yes)
+			)
+		)
+		(property "Value" "GND"
+			(at 21.59 53.34 0)
+			(effects
+				(font
+					(size 1.27 1.27)
+				)
+				(hide yes)
+			)
+		)
+		(property "Footprint" ""
+			(at 21.59 48.26 0)
+			(effects
+				(font
+					(size 1.27 1.27)
+				)
+				(hide yes)
+			)
+		)
+		(property "Datasheet" ""
+			(at 21.59 48.26 0)
+			(effects
+				(font
+					(size 1.27 1.27)
+				)
+				(hide yes)
+			)
+		)
+		(property "Description" "Power symbol creates a global label with name \"GND\" , ground"
+			(at 21.59 48.26 0)
+			(effects
+				(font
+					(size 1.27 1.27)
+				)
+				(hide yes)
+			)
+		)
+		(pin "1"
+		)
+		(instances
+			(project "robotic_hand_pcb"
+				(path "/96df9010-a1f8-4419-aac0-9388de87cb21/6d226a0a-d50a-47f5-bbb2-5bf13499a56e"
+					(reference "#PWR0122")
+					(unit 1)
+				)
