File: robotic_hand_pcb_analog.kicad_sch (KiCad schematic)
At the start: 26 parts, among them J10 A3, J11 A4, J12 A5, J13 A6, J14 A7, J8 A1, J9 A2, U10 ACS712xLCTR-05B, U11 ACS712xLCTR-05B, U12 ACS712xLCTR-05B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

Commit message: Update PCB for ADS114S08 rework fixes, v0.2.0
Connections:
- net +5V: now also U8.30 (REFP0)
- net GND: now also U8.29 (REFN0)
- no-connect marks 2 -> 0
