File: robotic_hand_pcb.kicad_sch (KiCad schematic)
At the start: 43 parts, among them J1 2171750001, J2 TC2050-IDC, J4 UART, SW1 SPST, U1 LMR51430, U2 ld39150dt33-r, U3 TXB0104QPWRQ1, U4 STM32F446RET, Y1 8M

Commit message: Near complete routing, cleanup
Parts:
- removed H1, H2, H3, H4: M3, MountingHole:MountingHole_3.2mm_M3_Pad_Via, symbol Mechanical:MountingHole_Pad
- added H1, H2, H3, H4: M3, MountingHole:MountingHole_3.2mm_M3, symbol Mechanical:MountingHole
Connections:
- net M5_1: now also U4.33 (PB12); no longer U4.36 (PB15)
- net M5_2: now also U4.34 (PB13); no longer U4.35 (PB14)
- net M5_3: now also U4.35 (PB14); no longer U4.34 (PB13)
- net M5_4: now also U4.36 (PB15); no longer U4.33 (PB12)
- net TIM1_CH1_PWM: now also U3.5 (A4); no longer U3.2 (A1)
- net TIM1_CH1_PWM_{5V}: now also U3.10 (B4); no longer U3.13 (B1)

Commit message: Initial full PCB design, pass DRC
Parts:
- added J3: Battery, robotic_hand_pcb_connectors:battery, symbol Connector:Conn_01x02_Pin
- added J4: Battery, Connector_PinHeader_2.54mm:PinHeader_1x02_P2.54mm_Vertical, symbol Connector:Conn_01x02_Pin
- added TP1: TestPoint, TestPoint:TestPoint_Pad_D2.5mm, symbol Connector:TestPoint
- C1, C2: footprint Capacitor_SMD:C_0603_1608Metric -> Capacitor_SMD:C_0805_2012Metric
- C3, C4: footprint Capacitor_SMD:C_0603_1608Metric -> Capacitor_SMD:C_1210_3225Metric
- L1: footprint Resistor_SMD:R_0603_1608Metric -> robotic_hand_pcb_inductor:vishay_ihlp-2525cz
- renumbered J3 to J5, J4 to J6
Connections:
- net +5V: now also J4.2 (Pin_2)
- net GND: now also J3.1 (Pin_1), J4.1 (Pin_1)
- net BUCK_SW: now reaches C1.2, L1.1, U1.2 (SW)
- net V_{IN} renamed +VSUPPLY
- net +VSUPPLY: now also J3.2 (Pin_2), TP1.1
Other:
- note added: "5V Breakout"
- moved on the sheet: C2

Commit message: Fix conflicting GPIO EXTI4 usage
Connections:
- net EXTI4_TOF_INT is gone; now on net GPIO_TOF_XSHUT: U4.56 (PB4)
- net GPIO_TOF_XSHUT: no longer U4.57 (PB5)
- new net EXTI5_TOF_INT: U4.57 (PB5)

Commit message: Fix C4 value error and cleanup silkscreen
Parts:
- C4: value 44u -> 22u
- J4: value Battery -> 5V
