File: robotic_hand_pcb_leds.kicad_sch (KiCad schematic)
At the start: 2 parts, among them J5 WS2812B

Commit message: Initial full PCB design, pass DRC
Parts:
- renumbered J5 to J7
Changed lines of the file:
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@@
 		(shape input)
 		(at 41.91 39.37 180)
-		(fields_autoplaced yes)
 		(effects
 			(font
@@
 		(dnp no)
 		(fields_autoplaced yes)
-		(property "Reference" "J5"
+		(property "Reference" "J7"
 			(at 76.2 40.6399 0)
 			(effects
@@
 			(project "robotic_hand_pcb"
 				(path "/96df9010-a1f8-4419-aac0-9388de87cb21/778b6ab7-1162-4b51-a46c-fb76fabecb49"
-					(reference "J5")
+					(reference "J7")
 					(unit 1)
 				)
@@
 		(dnp no)
 		(fields_autoplaced yes)
-		(property "Reference" "#PWR051"
+		(property "Reference" "#PWR056"
 			(at 50.8 54.61 0)
 			(effects
@@
 			(project "robotic_hand_pcb"
 				(path "/96df9010-a1f8-4419-aac0-9388de87cb21/778b6ab7-1162-4b51-a46c-fb76fabecb49"
-					(reference "#PWR051")
+					(reference "#PWR056")
 					(unit 1)
 				)
@@
 		(on_board yes)
 		(dnp no)
-		(property "Reference" "#PWR048"
+		(property "Reference" "#PWR053"
 			(at 50.8 34.29 0)
 			(effects
@@
 			(project "robotic_hand_pcb"
 				(path "/96df9010-a1f8-4419-aac0-9388de87cb21/778b6ab7-1162-4b51-a46c-fb76fabecb49"
-					(reference "#PWR048")
+					(reference "#PWR053")
 					(unit 1)
 				)
@@
 		(dnp no)
 		(fields_autoplaced yes)
-		(property "Reference" "#PWR050"
+		(property "Reference" "#PWR055"
 			(at 68.58 52.07 0)
 			(effects
@@
 			(project "robotic_hand_pcb"
 				(path "/96df9010-a1f8-4419-aac0-9388de87cb21/778b6ab7-1162-4b51-a46c-fb76fabecb49"
-					(reference "#PWR050")
+					(reference "#PWR055")
 					(unit 1)
 				)
@@
 		(on_board yes)
 		(dnp no)
-		(property "Reference" "#PWR049"
+		(property "Reference" "#PWR054"
 			(at 67.31 34.29 0)
 			(effects
@@
 			(project "robotic_hand_pcb"
 				(path "/96df9010-a1f8-4419-aac0-9388de87cb21/778b6ab7-1162-4b51-a46c-fb76fabecb49"
-					(reference "#PWR049")
-					(unit 1)
-				)
+					(reference "#PWR054")
+					(unit 1)
+				)
